Commit message: [Feature] working simulation

File: description/gazebo_control.xacro (robot description, xacro)
@@ -2,20 +2,28 @@
 <robot xmlns:xacro="http://www.ros.org/wiki/xacro">
     <gazebo>
-        <plugin name="diff_drive" filename="libgazebo_ros_diff_drive.so">
-            <!-- Wheel Information -->
-            <left_joint>wheel1_joint wheel4_joint</left_joint>
-            <right_joint>wheel2_joint wheel3_joint</right_joint>
-            <wheel_separation>0.57</wheel_separation>
-            <wheel_diameter>0.150</wheel_diameter>
-            <!-- Limits -->
-            <max_wheel_torque>200</max_wheel_torque>
-            <max_wheel_acceleration>10.0</max_wheel_acceleration>
-            <!-- Output -->
-            <odometry_frame>odom</odometry_frame>
-            <robot_base_frame>base_link</robot_base_frame>
-            <publish_odom>true</publish_odom>
-            <publish_odom_tf>true</publish_odom_tf>
-            <publish_wheel_tf>true</publish_wheel_tf>
+  <!-- Gazebo Harmonic physics plugin -->
+<plugin filename="gz-sim-diff-drive-system" name="gz::sim::systems::DiffDrive">
+    <left_joint>wheel1_joint</left_joint>
+    <right_joint>wheel2_joint</right_joint>
+    <wheel_separation>0.57</wheel_separation>
+    <wheel_diameter>0.150</wheel_diameter>
+    <max_wheel_torque>200</max_wheel_torque>
+    <max_wheel_acceleration>10.0</max_wheel_acceleration>
+    <topic>cmd_vel</topic>
+    <odom_topic>odom</odom_topic>
+    <odom_frame>odom</odom_frame>
+    <robot_base_frame>base_link</robot_base_frame>
+</plugin>
+<plugin filename="gz-sim-joint-state-publisher-system" name="gz::sim::systems::JointStatePublisher">
+            <topic>joint_states</topic>
+            <joint_name>wheel1_joint</joint_name>
+            <joint_name>wheel2_joint</joint_name>
+            <joint_name>wheel3_joint</joint_name>
+            <joint_name>wheel4_joint</joint_name>
         </plugin>
+<!-- ROS2 Control plugin -->
+<!-- <plugin filename="gz_ros2_control-system" name="gz_ros2_control::GzROS2ControlPlugin">
+    <parameters>$(find articubot_one)/config/controllers.yaml</parameters>
+</plugin> -->
     </gazebo>
 </robot>

File: description/lidar.xacro (robot description, xacro)
@@ -1,31 +1,93 @@
 <?xml version="1.0"?>
 <robot xmlns:xacro="http://www.ros.org/wiki/xacro" >
+<gazebo reference="imu_link">
+        <sensor name="imu" type="imu">
+        <always_on>true</always_on>
+        <update_rate>200</update_rate>
+        <visualize>true</visualize>
+        <topic>imu</topic>
+        <enable_metrics>true</enable_metrics>
+        <gz_frame_id>imu_link</gz_frame_id>
+        </sensor>
+    </gazebo>
     <gazebo reference="laser_frame">
-        <material>Gazebo/Black</material>
-        <sensor name="laser" type="ray">
+        <sensor name="laser" type="gpu_lidar">
             <pose> 0 0 0 0 0 0 </pose>
-            <visualize>false</visualize>
+            <always_on>true</always_on>
+            <visualize>true</visualize>
             <update_rate>10</update_rate>
-            <ray>
+            <topic>scan</topic>
+            <gz_frame_id>laser_frame</gz_frame_id>
+            <lidar>
                 <scan>
                     <horizontal>
-                        <samples>360</samples>
-                        <min_angle>-3.14</min_angle>
-                        <max_angle>3.14</max_angle>
+                    <samples>720</samples>
+                    <resolution>1</resolution>
+                    <min_angle>-3.14</min_angle>
+                    <max_angle>3.14</max_angle>
                     </horizontal>
                 </scan>
                 <range>
-                    <min>0.3</min>
-                    <max>12</max>
+                    <min>0.05</min>
+                    <max>10.0</max>
+                    <resolution>0.01</resolution>
                 </range>
-            </ray>
-            <plugin name="laser_controller" filename="libgazebo_ros_ray_sensor.so">
-                <ros>
-                    <argument>~/out:=scan</argument>
-                </ros>
-                <output_type>sensor_msgs/LaserScan</output_type>
-                <frame_name>laser_frame</frame_name>
-            </plugin>
+                <noise>
+                    <type>gaussian</type>
+                    <mean>0.0</mean>
+                    <stddev>0.01</stddev>
+                </noise>
+                <frame_id>laser_frame</frame_id>
+            </lidar>
+            <always_on>1</always_on>
+            <visualize>true</visualize>
         </sensor>
     </gazebo>
+<!--
+  <sensor name="laser" type="lidar">
+    <pose>0 0 0 0 0 0</pose>
+    <update_rate>10</update_rate>
+    <ray>
+        <scan>
+            <horizontal>
+                <samples>360</samples>
+                <min_angle>-3.14</min_angle>
+                <max_angle>3.14</max_angle>
+            </horizontal>
+        </scan>
+        <range>
+            <min>0.3</min>
+            <max>12</max>
+        </range>
+    </ray>
+    <visualize>false</visualize>
+</sensor>
+<gazebo reference="laser_frame">
+  <sensor name="laser" type="gpu_lidar">
+    <topic>scan</topic>
+    <update_rate>10</update_rate>
+    <lidar>
+      <scan>
+        <horizontal>
+          <samples>360</samples>
+          <resolution>1</resolution>
+          <min_angle>-3.14159</min_angle>
+          <max_angle>3.14159</max_angle>
+        </horizontal>
+      </scan>
+      <range>
+        <min>0.12</min>
+        <max>10.0</max>
+        <resolution>0.01</resolution>
+      </range>
+      <noise>
+        <type>gaussian</type>
+        <mean>0.0</mean>
+        <stddev>0.01</stddev>
+      </noise>
+    </lidar>
+    <always_on>1</always_on>
+    <visualize>true</visualize>
+  </sensor>
+</gazebo> -->
 </robot>

File: description/robot.urdf.xacro (robot description, xacro)
@@ -4,10 +4,10 @@
     <xacro:arg name="sim_mode" default="false"/>
     <xacro:include filename="robot_core.xacro" />
-    <xacro:if value="$(arg use_ros2_control)">
-        <xacro:include filename="ros2_control.xacro" />
-    </xacro:if>
-    <xacro:unless value="$(arg use_ros2_control)">
+    <!-- <xacro:if value="$(arg use_ros2_control)"> -->
+        <!-- <xacro:include filename="ros2_control.xacro" /> -->
+    <!-- </xacro:if> -->
+    <!-- <xacro:unless value="$(arg use_ros2_control)"> -->
         <xacro:include filename="gazebo_control.xacro" />
-    </xacro:unless>
+    <!-- </xacro:unless> -->
     <xacro:include filename="lidar.xacro" />
 </robot>

File: description/robot_core.xacro (robot description, xacro)
@@ -32,14 +32,19 @@
       </material>
     </visual>
-    <collision>
-      <origin
-        xyz="0 0 0"
-        rpy="0 0 0" />
-      <geometry>
-        <mesh
-          filename="file://$(find articubot_one)/meshes/chassis.STL" />
-      </geometry>
-    </collision>
-  </link>
+<collision name="chassis_collision">
+  <geometry>
+    <box size="0.3 0.3 0.15"/>
+  </geometry>
+</collision>
+  </link>
+  <!-- IMU Link -->
+      <link name="imu_link">
+      </link>
+      <!-- IMU Joint (fixed to chassis) -->
+      <joint name="imu_joint" type="fixed">
+        <parent link="chassis"/>
+        <child link="imu_link"/>
+        <origin xyz="0 0 0.1" rpy="0 0 0"/>
+      </joint>
   <link
     name="wheel1">
@@ -64,21 +69,17 @@
       <geometry>
         <mesh
-		filename="file://$(find articubot_one)/meshes/wheel1.STL" />
-      </geometry>
-      <material
-        name="">
-        <color
-          rgba="0.79216 0.81961 0.93333 1" />
-      </material>
-    </visual>
-    <collision>
-      <origin
-        xyz="0 0 0"
-        rpy="0 0 0" />
-      <geometry>
-        <mesh
-          filename="file://$(find articubot_one)/meshes/wheel1.STL" />
-      </geometry>
-    </collision>
+    filename="file://$(find articubot_one)/meshes/wheel1.STL" />
+      </geometry>
+      <material
+        name="">
+        <color
+          rgba="0.79216 0.81961 0.93333 1" />
+      </material>
+    </visual>
+<collision name="wheel1_collision">
+  <geometry>
+    <cylinder radius="0.1" length="0.05"/>
+  </geometry>
+</collision>
   </link>
   <joint name="base_footprint_to_chassis" type="fixed">
@@ -91,5 +92,5 @@
     type="continuous">
     <origin
-      xyz="0.23 -0.285 -0.2"
+      xyz="0.23 -0.285 -0.25"
       rpy="-1.5708 0 0" />
     <parent
@@ -99,9 +100,5 @@
     <axis
       xyz="0 0 1" />
-    <limit
-      lower="60"
-      upper="45"
-      effort="7.6"
-      velocity="5.24" />
+    <limit effort="1000.0" velocity="20.0" />
     <dynamics
       damping="0.2"
@@ -138,13 +135,9 @@
       </material>
     </visual>
-    <collision>
-      <origin
-        xyz="0 0 0"
-        rpy="0 0 0" />
-      <geometry>
-        <mesh
-          filename="file://$(find articubot_one)/meshes/wheel2.STL" />
-      </geometry>
-    </collision>
+    <collision name="wheel2_collision">
+  <geometry>
+    <cylinder radius="0.1" length="0.05"/>
+  </geometry>
+</collision>
   </link>
   <joint
@@ -152,5 +145,5 @@
     type="continuous">
     <origin
-      xyz="-0.23 -0.285 -0.2"
+      xyz="-0.23 -0.285 -0.25"
       rpy="-1.5708 0 0" />
     <parent
@@ -160,4 +153,5 @@
     <axis
       xyz="0 0 1" />
+    <limit effort="1000.0" velocity="20.0" />
   </joint>
   <link
@@ -191,15 +185,11 @@
       </material>
     </visual>
-    <collision>
-      <origin
-        xyz="0 0 0"
-        rpy="0 0 0" />
-      <geometry>
-        <mesh
-		filename="file://$(find articubot_one)/meshes/wheel3.STL" />
-      </geometry>
-    </collision>
-  </link>
-  <joint
+  <collision name="wheel3_collision">
+  <geometry>
+    <cylinder radius="0.1" length="0.05"/>
+  </geometry>
+</collision>
+  </link>
+<joint
     name="wheel3_joint"
     type="continuous">
@@ -244,13 +234,9 @@
       </material>
     </visual>
-    <collision>
-      <origin
-        xyz="0 0 0"
-        rpy="0 0 0" />
-      <geometry>
-        <mesh
-          filename="file://$(find articubot_one)/meshes/wheel4.STL" />
-      </geometry>
-    </collision>
+   <collision name="wheel4_collision">
+  <geometry>
+    <cylinder radius="0.1" length="0.05"/>
+  </geometry>
+</collision>
   </link>
   <joint
@@ -258,5 +244,5 @@
     type="continuous">
     <origin
-      xyz="-0.23 0.285 -0.2"
+      xyz="-0.23 0.285 -0.25"
       rpy="-1.5708 0 0" />
     <parent
@@ -266,4 +252,5 @@
     <axis
       xyz="0 0 -1" />
+   <limit effort="1000.0" velocity="20.0" />
   </joint>
   <link
@@ -297,13 +284,9 @@
       </material>
     </visual>
-    <collision>
-      <origin
-        xyz="0 0 0"
-        rpy="0 0 0" />
-      <geometry>
-        <mesh
-          filename="file://$(find articubot_one)/meshes/lidar.STL" />
-      </geometry>
-    </collision>
+  <collision name="laser_frame_collision">
+  <geometry>
+    <cylinder radius="0.1" length="0.05"/>
+  </geometry>
+</collision>
   </link>
   <joint

File: description/ros2_control.xacro (robot description, xacro)
@@ -31,8 +31,8 @@
         </ros2_control>
     </xacro:unless>
-    <xacro:if value="$(arg sim_mode)">
+    <!-- <xacro:if value="$(arg sim_mode)"> -->
         <ros2_control name="GazeboSystem" type="system">
             <hardware>
-                <plugin>gazebo_ros2_control/GazeboSystem</plugin>
+                <plugin>gz_ros2_control/GazeboSimSystem</plugin>
             </hardware>
             <joint name="wheel1_joint">
@@ -69,9 +69,9 @@
             </joint>
         </ros2_control>
-    </xacro:if>
+    <!-- </xacro:if> -->
     <gazebo>
-        <plugin name="gazebo_ros2_control" filename="libgazebo_ros2_control.so">
+       <plugin filename="gz_ros2_control-system" name="gz_ros2_control::GazeboSimROS2ControlPlugin">
             <parameters>$(find articubot_one)/config/my_controllers.yaml</parameters>
-            <parameters>$(find articubot_one)/config/gaz_ros2_ctl_use_sim.yaml</parameters>
+            <!-- <parameters>$(find articubot_one)/config/gaz_ros2_ctl_use_sim.yaml</parameters> -->
         </plugin>
     </gazebo>
